Commit message: Mejor pista

File: puzzlebot_gazebo/urdf/puzzlebot.xacro (robot description, xacro)
@@ -155,5 +155,5 @@
 	  <parent link="chassis" />
 	  <child link="camera" />
-	  <origin xyz="0.09 0 0.048" />
+	  <origin xyz="0.11 0 0.048" rpy = "0 ${PI/4} 0"/>
   </joint>
 <!-- TRANSMISSIONS (For a more complex model and it represents actuator attributes) -->
